File: Battery Featherwing.kicad_pcb (KiCad board)
At the start: 2 copper layers, 23.4 x 51.3 mm, 39 parts, among them J1 Battery, J2 Neopix A, J3 Neopix B, U1 INA3221, U2 TPS61090, U3 MCP73871, U4 MAX17048G_T10, U5 74AUC2G07

Commit message: Added some text to the board, for practice.
Other:
- board text added: "Bad Mink Things"
Changed lines of the file:
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@@
 		(fp_arc
 			(start -1.52 -3.81)
-			(mid -0.702828 -5.782827)
+			(mid -0.702828 -5.782828)
 			(end 1.27 -6.6)
 			(stroke
@@
 		)
 	)
+	(gr_text "Bad Mink Things"
+		(at 110.109 77.089 0)
+		(layer "F.SilkS")
+		(effects
+			(font
+				(size 1.5 1.5)
+				(thickness 0.1875)
+			)
+			(justify left bottom)
+		)
+	)
